File: MercuryBase_4slot.kicad_pcb (KiCad board)
At the start: 2 copper layers, 124 x 108 mm, 106 parts, among them IC201 AP62200WU-7, J1 Conn_01x02, J10 Conn_01x03, J101 Conn_01x02_Pin, J11 Conn_01x06, J14 Conn_02x15_Odd_Even, J15 Conn_02x15_Odd_Even, J16 MC-802YC-H105, J2 Conn_02x15_Odd_Even, J201 Mini360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

Commit message: first
Parts:
- removed C12: 10uF/50V, Capacitor_SMD:C_0805_2012Metric
- removed D3: CESDLC5V0M5, Package_TO_SOT_SMD:SOT-563
- removed IC201: AP62200WU-7, Package_TO_SOT_SMD:SOT95P280X100-6N
- removed J16: MC-802YC-H105, uSB:MC-802YC-H105
- removed R10: 100R, Resistor_SMD:R_0603_1608Metric
- removed R11: 47,5K, Resistor_SMD:R_0603_1608Metric
- removed R12: 1K, Resistor_SMD:R_0603_1608Metric
- removed R13: 10K, Resistor_SMD:R_0603_1608Metric
- removed R301, R302: 5,1K, Resistor_SMD:R_0603_1608Metric
- removed R9: 22K, Resistor_SMD:R_0603_1608Metric
- removed U4: CP2102N-Axx-xQFN24, Package_DFN_QFN:QFN-24-1EP_4x4mm_P0.5mm_EP2.6x2.6mm
- added IC1: AOZ1283PI, Package_SO:Diodes_SO-8EP, F.Cu at (54.2, 57.6)
- added J7: Conn_02x05_Odd_Even, Connector_PinHeader_2.54mm:PinHeader_2x05_P2.54mm_Vertical, F.Cu at (62.6, 137.3)
- added R6: 20K, Resistor_SMD:R_0603_1608Metric, F.Cu at (49.6, 52.9)
- C10: value 10uF/50V -> 100nF/50V; footprint Capacitor_SMD:C_0805_2012Metric -> Capacitor_SMD:C_0603_1608Metric
- C11: value 100nF/50V -> 33uF/50V; footprint Capacitor_SMD:C_0603_1608Metric -> Capacitor_SMD:CP_Elec_6.3x7.7
- C3: value 330uF 35V -> 33uF/50V; footprint Capacitor_SMD:CP_Elec_10x10.5 -> Capacitor_SMD:CP_Elec_6.3x7.7
- C4: value 22uF/25V -> 4,7uF/50V
- C9: value 100nF/50V -> 1nF; footprint Capacitor_SMD:C_0603_1608Metric -> Capacitor_SMD:C_0805_2012Metric
- D1: value SS210 -> SS56F-DC
- D2: value LED -> SS56F-DC; footprint LED_SMD:LED_0805_2012Metric -> Diode_SMD:D_SMA
- L1: value 4,7uH -> 22uH; footprint Inductor_SMD:L_TracoPower_TCK-047_5.2x5.8mm -> Inductor_SMD:L_12x12mm_H6mm
- R8: value 4,7K -> 100K
- moved R202 85.4 mm to (72.9, 139.4), turned to -90 degrees
- moved C9 83.2 mm to (51.7, 52.9)
- moved C11 82.4 mm to (67.5, 44.7)
- moved D6 81.9 mm to (72.9, 136.1), turned to 90 degrees
- moved J101 80.9 mm to (52.8, 136.6), turned to 180 degrees
- moved R8 78.8 mm to (56.7, 52.9), turned to 90 degrees
- moved D2 77.2 mm to (61.2, 57.9)
- moved C10 75.1 mm to (52.4, 61.3), turned to 0 degrees
- moved J1 72.3 mm to (55.2, 114.0)
- moved C7 31.3 mm to (80.5, 56.0)
- moved L1 16.8 mm to (71.7, 56.1), turned to 0 degrees
- moved R19 15.4 mm to (48.3, 62.0), turned to 180 degrees
- moved R21 12.6 mm to (48.3, 60.0), turned to 0 degrees
- moved D4 9.68 mm to (85.9, 46.6)
- moved D5 9.68 mm to (85.9, 48.9)
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Connections:
- C10 pad 1: Net-(D3-IO3) -> Net-(IC1-SS)
- C10 pad 2: GND -> +12V
- C11 pad 1: Net-(U4-VDD) -> +12V
- C3 pad 1: +12V -> +5V
- C5 pad 1: Net-(IC201-SW) -> Net-(D2-K)
- C9 pad 1: Net-(D3-IO3) -> Net-(C9-Pad1)
- C9 pad 2: GND -> Net-(IC1-COMP)
- D2 pad 1: GND -> Net-(D2-K)
- D2 pad 2: Net-(D2-A) -> GND
- J10 pad 3: /USB/RXD -> /USB/TXD
- J9 pad 3: /USB/TXD -> /USB/RXD
- L1 pad 1: Net-(IC201-SW) -> Net-(D2-K)
- R8 pad 1: Net-(D3-IO3) -> Net-(IC1-FSW)
- R8 pad 2: Net-(D2-A) -> GND
Routing:
- net GND: track 129.9 -> 175.7 mm, vias 17 -> 20
- net Net-(D3-IO3): track 39.3 -> 0.00 mm
- net +12V: track 331.1 -> 360.0 mm
- net Net-(U4-VDD): track 19.8 -> 0.00 mm, vias 2 -> 0
- net /IO18: track 396.2 -> 378.5 mm
- net /IO0: track 332.2 -> 314.6 mm
- net Net-(D2-K): track 0.00 -> 11.9 mm
- net Net-(D3-IO2): track 10.4 -> 0.00 mm, vias 2 -> 0
- net Net-(D3-IO1): track 9.57 -> 0.00 mm
- net /IO19: track 403.4 -> 394.5 mm
- net Net-(J16-CC1): track 7.93 -> 0.00 mm, vias 1 -> 0
- net Net-(J16-CC2): track 6.83 -> 0.00 mm, vias 1 -> 0
- net +3.3V: track 355.5 -> 350.0 mm, vias 7 -> 6
- net Net-(IC1-SS): track 0.00 -> 5.33 mm
- net Net-(U4-~{RST}): track 5.08 -> 0.00 mm
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- added copper zone on B.Cu, net +12V
- removed copper zone on B.Cu, net Net-(IC201-SW)
- removed copper zone on F.Cu, net Net-(IC201-SW)
Other:
- board text added: "3V3"
- board text added: "DTR-IO0"
- board text added: "G N D"
- board text added: "MERCURY 1.1.0"
- board text added: "RTS-EN"
- board text added: "RXD"
- board text added: "TCK"
- board text added: "TDI"
- board text added: "TDO"
- board text added: "TMS"
- board text added: "TXD"
- board text removed: "MERCURY 1.0.0"
