File: MercuryBase_4slot.kicad_sch (KiCad schematic)
At the start: 20 parts, among them J1 Conn_01x02, J10 Conn_01x03, J101 Conn_01x02_Pin, J11 Conn_01x06, J14 Conn_02x15_Odd_Even, J15 Conn_02x15_Odd_Even, J2 Conn_02x15_Odd_Even, J3 Conn_02x15_Odd_Even, J4 Conn_02x05_Odd_Even, J5 Conn_01x02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

Commit message: first
Parts:
- C1, C2: value 100nF/50V -> 100nF/16V; Cena (none) -> 0,03; TME (none) -> CC0603KRX7R7BB104
- J1, J5, J6: Cena (none) -> 0,03
- J10, J9: Cena (none) -> 0,06; MARITEX (none) -> PLS40S-CT
- J101: Cena (none) -> 0,04; MARITEX (none) -> PLS40S-CT
- J11: Cena (none) -> 0,12; MARITEX (none) -> PLS40S-CT
- J14: Cena (none) -> 1,45; MARITEX (none) -> PBD30S-CT; now in the parts list
- J15, J2, J3: Cena (none) -> 1,45; MARITEX (none) -> PBD30S-CT
- J4: value Conn_02x05_Odd_Even -> Conn_02x05_Odd_Male; Cena (none) -> 0,25; MARITEX (none) -> PLD10SU
- R1: Cena (none) -> 0,01; TME (none) -> SMD0603-10K-1%
- R2, R3, R4, R5: Cena (none) -> 0,01; TME (none) -> SMD0805-100R-1%
- U1: Cena (none) -> 20,91; SOSelectronic (none) -> 287426
Connections:
- net USB/RXD: now also J9.3 (Pin_3); no longer J10.3 (Pin_3)
- net USB/TXD: now also J10.3 (Pin_3); no longer J9.3 (Pin_3)
Other:
- moved on the sheet: C1, C2, J101, J14, J15, J2, J3, R1, U1
