File: POWER.kicad_sch (KiCad schematic)
At the start: 22 parts, among them IC201 AP62200WU-7, J201 Mini360, P1 CONN_01X02, U2 AP62200Z6-7, U3 AMS1117-3.3

Commit message: first
Parts:
- removed C3: 330uF 35V, Capacitor_SMD:CP_Elec_10x10.5, symbol felisiak01-rescue:CP-device
- removed IC201: AP62200WU-7, Package_TO_SOT_SMD:SOT95P280X100-6N, symbol Regulator_Switching:AP62200WU-7
- removed U2: AP62200Z6-7, Package_TO_SOT_SMD:SOT-563, symbol Regulator_Switching:AP62150Z6
- added C10: 100nF/50V, Capacitor_SMD:C_0603_1608Metric, symbol Device:C
- added C11: 100uF/35V, Capacitor_SMD:CP_Elec_6.3x7.7, symbol B800_2-rescue:CP_Small-device
- added C3: 100uF/6,3V, Capacitor_SMD:CP_Elec_6.3x7.7, symbol B800_2-rescue:CP_Small-device
- added C9: 1nF, Capacitor_SMD:C_0805_2012Metric, symbol Device:C
- added D2: SS56F-DC, Diode_SMD:D_SMA, symbol felisiak01-rescue:D-device
- added IC1: AOZ1283PI, Package_SO:Diodes_SO-8EP, symbol Regulator_Switching:AOZ1283PI
- added P2: 15EDGK-3.5-02P-14-00Z(H), Connector_Phoenix_MC:PhoenixContact_MCV_1,5_2-G-3.5_1x02_P3.50mm_Vertical, symbol felisiak01-rescue:CONN_01X02-conn
- added R6: 20K, Resistor_SMD:R_0603_1608Metric, symbol felisiak01-rescue:R_Small-device
- added R8: 100K, Resistor_SMD:R_0603_1608Metric, symbol felisiak01-rescue:R_Small-device
- C4: value 22uF/25V -> 4,7uF/35V; Cena (none) -> 0,4; TME (none) -> GRT21BC8YA475KE13L
- C5: Cena (none) -> 0,01; TME (none) -> 0603B104K500CT
- C6, C7: value 22uF/25V -> 22uF/10V; Cena (none) -> 0,26; TME (none) -> 0805X226M100CT
- C8: value 100nF/50V -> 100nF/16V; Cena (none) -> 0,03; TME (none) -> CC0603KRX7R7BB104
- D1: value SS210 -> SS56F-DC; Cena (none) -> 0,4; TME (none) -> SS56F-DC
- L1: value 4,7uH -> 22uH; footprint Inductor_SMD:L_TracoPower_TCK-047_5.2x5.8mm -> Inductor_SMD:L_12x12mm_H6mm; Cena (none) -> 1,3; LCSC part# C405142 -> (none); TME (none) -> DE1205-22
- P1: Cena (none) -> 0,4; MARITEX (none) -> KF2EDGV-Y-3.50-2P; now in the parts list
- R16, R7: Cena (none) -> 0,01; TME (none) -> SMD0603-10K-1%
- R19: Cena (none) -> 0,01; TME (none) -> 0603SAJ0513T5E
- R201: Cena (none) -> 0,01; TME (none) -> 0603SAF2701T5E
- R202: Cena (none) -> 0,01; TME (none) -> 0603SAF1801T5E
- R21: value 1,2K -> 1,3K; Cena (none) -> 0,01; TME (none) -> 0603SAF1301T5E
- U3: Cena (none) -> 0,54; TME (none) -> LDI1117-3.3H-DIO
Connections:
- net 12V: now also C10.2, C11.1, IC1.9 (VIN)
- net 5V: now also C3.1
- net GND: now also C11.2, C3.2, D2.2 (A), IC1.3 (GND), R6.2, R8.2
- net at R21.2, R7.1: now also IC1.6 (FB)
- net at C5.1, L1.1: now also D2.1 (K), IC1.1 (LX)
- net at C5.2: now also IC1.2 (BST)
- new net: C10.1, IC1.7 (SS)
- new net: IC1.4 (FSW), R8.1
- new net: C9.2, IC1.5 (COMP)
- new net: C9.1, R6.1
Other:
- note added: "52,2"
- note added: "zmienić na 0603 RF-GSB190TS-BC"
- moved on the sheet: C5, L1
