File: USB.kicad_sch (KiCad schematic)
At the start: 20 parts, among them J16 MC-802YC-H105, Q1 SS8050, Q2 SS8050, U4 CP2102N-Axx-xQFN24

Commit message: first
Parts:
- removed C10, C12: 10uF/50V, Capacitor_SMD:C_0805_2012Metric, symbol Device:C
- removed C11, C9: 100nF/50V, Capacitor_SMD:C_0603_1608Metric, symbol Device:C
- removed D2: LED, LED_SMD:LED_0805_2012Metric, symbol Device:LED
- removed D3: CESDLC5V0M5, Package_TO_SOT_SMD:SOT-563, symbol Power_Protection:ESDA6V1-5SC6
- removed J16: MC-802YC-H105, uSB:MC-802YC-H105, symbol USB:MC-802YC-H105
- removed R10: 100R, Resistor_SMD:R_0603_1608Metric, symbol Device:R
- removed R11: 47,5K, Resistor_SMD:R_0603_1608Metric, symbol Device:R
- removed R12: 1K, Resistor_SMD:R_0603_1608Metric, symbol Device:R
- removed R13: 10K, Resistor_SMD:R_0603_1608Metric, symbol Device:R
- removed R301, R302: 5,1K, Resistor_SMD:R_0603_1608Metric, symbol Device:R
- removed R8: 4,7K, Resistor_SMD:R_0603_1608Metric, symbol Device:R
- removed R9: 22K, Resistor_SMD:R_0603_1608Metric, symbol Device:R
- removed U4: CP2102N-Axx-xQFN24, Package_DFN_QFN:QFN-24-1EP_4x4mm_P0.5mm_EP2.6x2.6mm, symbol Interface_USB:CP2102N-Axx-xQFN24
- added J7: Conn_02x05_Odd_Female, Connector_PinHeader_2.54mm:PinHeader_2x05_P2.54mm_Vertical, symbol Connector_Generic:Conn_02x05_Odd_Even
- Q1, Q2: Cena (none) -> 0,054; TME (none) -> BC817-16-YAN
- R14, R15: value 12K -> 10K; Cena (none) -> 0,01; TME (none) -> SMD0603-10K-1%
Connections:
- net DTR: now also J7.10 (Pin_10)
- net GND: now also J7.5 (Pin_5)
- net RTS: now also J7.8 (Pin_8)
- net RXD: now also J7.9 (Pin_9)
- net TXD: now also J7.7 (Pin_7)
- new net: J7.4 (Pin_4), J7.6 (Pin_6)
Other:
- note added: "Jumper 3V3"
- note added: "USB"
- note added: "USB3v3"
- note added: "USB5V"
- moved on the sheet: Q1, Q2, R14, R15
